File: PCB/cup_sense/cup_sense.kicad_sch (KiCad schematic)
At the start: 36 parts, among them J1 Connect, J2 Connect, J3 Connect, J4 Connect, J5 Connect, J6 Connect, J7 UPDI, Q1 Q_Photo_NPN, Q2 BC847, Q3 BC847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

Commit message: v1.0
Parts:
- J1, J2, J6: footprint fsr:1x09_EdgeConnect -> fsr:1x09_EdgeConnect_Flip
Connections:
- net LED_IN: now also J1.2 (Pin_2), J2.2 (Pin_2), J6.2 (Pin_2); no longer J1.3 (Pin_3), J2.3 (Pin_3), J6.3 (Pin_3)
- net LED_OUT: now also J1.3 (Pin_3), J2.3 (Pin_3), J6.3 (Pin_3); no longer J1.2 (Pin_2), J2.2 (Pin_2), J6.2 (Pin_2)
Other:
- note added: "10k"
- moved on the sheet: J1, J2, J3, J4, J5, J6

Commit message: fix schematic values
Other:
- note added: "1M"
- note removed: "10k"
- moved on the sheet: J1, J2, J3, J4, J5, J6
